File: Aux.kicad_sch (KiCad schematic)
At the start: 99 parts, among them T200 BC337, T301 BC328

Commit message: Add files via upload
Other:
- note added: "Pg 4 of 4"
- moved on the sheet: R302, R305, R306, R321, T200
