File: Dist-MPS.kicad_sch (KiCad schematic)
At the start: 90 parts, among them T200 BC337, T201 BC337, T260 BC337, T300 BC337, T301 BC328, T500 BC338, T501 BC337, T502 BC328, T503 BC328, T504 BC337, T505 BC338, T700 BC338, T701 BC338

Commit message: Add files via upload
Parts:
- added R318: 33k, symbol Device:R
- added R319: 110k, symbol Device:R
Connections:
- net BRN: now also R318.1, R319.1; no longer R240.2
- net MPS (7): now also R224.2, T201.1 (C)
- net Fuel Pump ON: now reaches D500.2 (A), R509.2, T501.3 (E), T504.3 (E)
- new net MPS (10): R240.2, R318.2, R319.2
Other:
- note added: "Pg 2 of 4"
- moved on the sheet: C200, C201, C209, C212, C500, C501, C700, D201, D203, D204, D205, D206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
