File: ECU Conn.kicad_sch (KiCad schematic)
At the start: 32 parts, among them J1 Conn_01x04_Pin, J10 Conn_01x04_Pin, J11 Conn_01x03_Pin, J12 Conn_01x03_Socket, J13 Conn_01x04_Socket, J14 Conn_01x04_Pin, J15 Conn_01x02_Socket, J16 Conn_01x02_Socket, J17 Conn_01x02_Socket, J18 Conn_01x02_Socket, J19 Conn_01x02_Socket, J2 Conn_01x04_Socket, J20 Conn_01x02_Socket, J21 Conn_01x02_Pin, J22 Conn_01x02_Pin, J27 Conn_01x07_Pin, J28 Conn_01x07_Socket, J3 Conn_01x03_Pin, J4 Conn_01x03_Pin, J5 Conn_01x03_Socket, J6 Conn_01x03_Socket, J7 Conn_01x04_Socket, J8 Conn_01x04_Socket, J9 Conn_01x04_Socket, K1 Fuel Injection Main Relay, K2 Fuel Pump Relay, SW1 SW_SPST, SW2 SW_SPST

Commit message: Add files via upload
Other:
- note added: "Pg 1 of 4"
- moved on the sheet: TS1-Air, TS2-Coolant, Vacuum
