File: TPS.kicad_sch (KiCad schematic)
At the start: 104 parts, among them T200 BC337, T301 BC328

Commit message: Add files via upload
Parts:
- R406: value R? -> 1k
Connections:
- net at R518.1: now also C907.2, D903.2 (A), R911.2, T200.1 (C)
- net Fuel Pump ON: now reaches D403.1 (K)
Other:
- note added: "Pg 3 of 4"
- moved on the sheet: C301, C302, C902, C906, C907, D301, D302, D303, D305, D308, D402, D908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
